File: idc40_breakout.kicad_pcb (KiCad board)
At the start: 2 copper layers, 17.3 x 104.1 mm, 2 parts, among them J1 Conn_01x40, J2 Conn_01x40

Commit message: Update for KiCad 6
Other:
- net class Default removed
